File: pcb/tiny-vga.kicad_sch (KiCad schematic)
At the start: 13 parts, among them J1 PMOD, J2 VGA, U1 74LVC245A

Commit message: Update parts for aisler
Parts:
- removed C1: C, Capacitor_SMD:C_0603_1608Metric_Pad1.08x0.95mm_HandSolder, symbol Device:C_Small
- removed JP1: SolderJumper_3_Bridged12, Jumper:SolderJumper-3_P1.3mm_Bridged2Bar12_RoundedPad1.0x1.5mm, symbol Jumper:SolderJumper_3_Bridged12
- J1: MPN (none) -> 826634-6
- J2: MPN (none) -> L77HDE15SD1CH4FVGA
- R1, R2, R3: MPN (none) -> CR0402-FX-3600GLF
- R4, R5: MPN (none) -> RK73H1ETTP47R0F
- RN1, RN2, RN3: footprint Resistor_SMD:R_Array_Convex_4x0402 -> Resistor_SMD:R_Array_Convex_4x0603; MPN (none) -> CAY16-361J4LF
- U1: value 74LVC245A -> 74LVC245APW,118; MPN (none) -> 74LVC245APW,118
Connections:
- net GND: now also U1.1 (DIR)

Commit message: Add AISLER support
Parts:
- removed R1, R2, R3: 360R, Resistor_SMD:R_0402_1005Metric, symbol Device:R
- removed RN1, RN2, RN3: 360R, Resistor_SMD:R_Array_Convex_4x0603, symbol Device:R_Pack04_Split
- added C1: 100n, Capacitor_SMD:C_0603_1608Metric, symbol Device:C_Small
- added R1, R11, R16, R17, R19, R24, R3, R8, R9: 470, Resistor_SMD:R_0402_1005Metric, symbol Device:R_Small
- added R10, R13, R15, R18, R2, R21, R23, R5, R7: 1.5k, Resistor_SMD:R_0402_1005Metric, symbol Device:R_Small
- added R12, R20, R4: 220R, Resistor_SMD:R_0402_1005Metric, symbol Device:R_Small
- added R14, R22, R6: 1k, Resistor_SMD:R_0402_1005Metric, symbol Device:R_Small
- R25: renamed from R4; value 47R -> 49.9R; MPN RK73H1ETTP47R0F -> ERJ-2RKF49R9X
- R26: renamed from R5; value 47R -> 49.9R; MPN RK73H1ETTP47R0F -> ERJ-2RKF49R9X
Connections:
- net +3.3V: now also C1.1
- net AnalogB: now also R19.2, R20.2, R21.2, R22.2
- net AnalogG: now also R11.2, R12.2, R13.2, R14.2
- net AnalogR: now also R3.2, R4.2, R5.2, R6.2
- net B0: now also R23.1, R24.1
- net B1: now also R19.1, R21.1
- net G0: now also R15.1, R16.1
- net G1: now also R11.1, R13.1
- net GND: now also C1.2, R1.2, R10.2, R17.2, R18.2, R2.2, R9.2
- net R0: now also R7.1, R8.1
- net R1: now also R3.1, R5.1
- new net: R1.1, R2.1, R4.1, R6.1, R7.2, R8.2
- new net: R17.1, R18.1, R20.1, R22.1, R23.2, R24.2
- new net: R10.1, R12.1, R14.1, R15.2, R16.2, R9.1
