File: pcb/tiny-vga.kicad_sch (KiCad schematic)
At the start: 30 parts, among them J1 PMOD, J2 VGA, U1 74LVC245APW,118

Commit message: Final v1.2, tested and working
Parts:
- J2: footprint tiny-vga:DSUB-15-HD_Female_Horizontal -> Connector_Dsub:DSUB-15-HD_Female_Horizontal_P2.29x1.98mm_EdgePinOffset8.35mm_Housed_MountingHolesOffset10.89mm

Commit message: Update to KiCad 8.0
Parts:
- C1: LCSC (none) -> C14663
- J1: LCSC (none) -> C2935938
- J2: LCSC (none) -> C138387
- R1, R11, R16, R17, R19, R24, R3, R8, R9: LCSC (none) -> C25117
- R10, R13, R15, R18, R2, R21, R23, R5, R7: LCSC (none) -> C25867
- R12, R20, R4: LCSC (none) -> C25091
- R14, R22, R6: LCSC (none) -> C11702
- R25, R26: LCSC (none) -> C25120
- U1: LCSC (none) -> C6082
Other:
- note added: "75 Ω termination"
- note added: "Pmod"
- note removed: "PMOD"
- moved on the sheet: U1
