File: pcb/tiny-vga.kicad_pcb (KiCad board)
At the start: 2 copper layers, 40 x 33 mm, 32 parts, among them J1 PMOD, J2 VGA, U1 74LVC245APW,118

Commit message: Final v1.2, tested and working
Parts:
- J2: footprint tiny-vga:DSUB-15-HD_Female_Horizontal -> tiny-vga:VGA-002
- moved J2 0.30 mm to (160.0, 73.2)
Routing:
- net AnalogB: track 11.9 -> 12.7 mm
- net Net-(J2-Pad14): track 17.7 -> 18.3 mm
